Commit message: updated urdf for ur5e arm with robotiq 2f 140 gripper

File: source/isaaclab_assets/data/ur5e_dual_setup/ur5e_robotiq_2f_140.urdf (robot description, URDF)
Before this commit: robot ur5e, 13 links, 12 joints
Links:
- removed link base
- removed link base_link
- removed link flange
- removed link robotiq_arg2f_base_link
- removed link tool0
- added link ee_link_robotiq_arg2f_base_link, mass 0.22652; collision mesh filename=file:///home/till/IsaacLab/source/isaaclab_assets/data/ur5e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 scale=1. 1. 1.; visual mesh filename=file:///home/till/IsaacLab/source/isaaclab_assets/data/ur5e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 scale=1. 1. 1.
- added link left_inner_finger, mass 0.0104003; collision box size=0.03 0.07 0.0075; collision mesh filename=file:///home/till/IsaacLab/source/isaaclab_assets/data/ur5e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 scale=1. 1. 1.
- added link left_inner_knuckle, mass 0.0271177; collision mesh filename=file:///home/till/IsaacLab/source/isaaclab_assets/data/ur5e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 scale=1. 1. 1.; visual mesh filename=file:///home/till/IsaacLab/source/isaaclab_assets/data/ur5e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 scale=1. 1. 1.
- added link left_outer_finger, mass 0.0226142; collision mesh filename=file:///home/till/IsaacLab/source/isaaclab_assets/data/ur5e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 scale=1. 1. 1.; visual mesh filename=file:///home/till/IsaacLab/source/isaaclab_assets/data/ur5e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 scale=1. 1. 1.
- added link left_outer_knuckle, mass 0.008532; collision mesh filename=file:///home/till/IsaacLab/source/isaaclab_assets/data/ur5e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 scale=1. 1. 1.; visual mesh filename=file:///home/till/IsaacLab/source/isaaclab_assets/data/ur5e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 scale=1. 1. 1.
- added link right_inner_finger, mass 0.0104003; collision box size=0.03 0.07 0.0075; collision mesh filename=file:///home/till/IsaacLab/source/isaaclab_assets/data/ur5e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 scale=1. 1. 1.
- added link right_inner_knuckle, mass 0.0271177; collision mesh filename=file:///home/till/IsaacLab/source/isaaclab_assets/data/ur5e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 scale=1. 1. 1.; visual mesh filename=file:///home/till/IsaacLab/source/isaaclab_assets/data/ur5e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 scale=1. 1. 1.
- added link right_outer_finger, mass 0.0226142; collision mesh filename=file:///home/till/IsaacLab/source/isaaclab_assets/data/ur5e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 scale=1. 1. 1.; visual mesh filename=file:///home/till/IsaacLab/source/isaaclab_assets/data/ur5e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 scale=1. 1. 1.
- added link right_outer_knuckle, mass 0.008532; collision mesh filename=file:///home/till/IsaacLab/source/isaaclab_assets/data/ur5e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 scale=1. 1. 1.; visual mesh filename=file:///home/till/IsaacLab/source/isaaclab_assets/data/ur5e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 scale=1. 1. 1.
- added link ur
- added link world
- link base_link_inertia: mass 4.0 -> 4.; geometry collision mesh filename=file:///home/till/IsaacLab/source/isaaclab_assets/data/ur5e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 scale=1. 1. 1.; visual mesh filename=file:///home/till/IsaacLab/source/isaaclab_assets/data/ur5e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 scale=1. 1. 1.
- link forearm_link: mass 2.275 -> 2.846; geometry collision mesh filename=file:///home/till/IsaacLab/source/isaaclab_assets/data/ur5e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 scale=1. 1. 1.; visual mesh filename=file:///home/till/IsaacLab/source/isaaclab_assets/data/ur5e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 scale=1. 1. 1.
- link shoulder_link: mass 3.7 -> 3.7609999; geometry collision mesh filename=file:///home/till/IsaacLab/source/isaaclab_assets/data/ur5e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 scale=1. 1. 1.; visual mesh filename=file:///home/till/IsaacLab/source/isaaclab_assets/data/ur5e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 scale=1. 1. 1.
- link upper_arm_link: mass 8.393 -> 8.0579996; geometry collision mesh filename=file:///home/till/IsaacLab/source/isaaclab_assets/data/ur5e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 scale=1. 1. 1.; visual mesh filename=file:///home/till/IsaacLab/source/isaaclab_assets/data/ur5e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 scale=1. 1. 1.
- link wrist_1_link: mass 1.219 -> 1.37; geometry collision mesh filename=file:///home/till/IsaacLab/source/isaaclab_assets/data/ur5e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 scale=1. 1. 1.; visual mesh filename=file:///home/till/IsaacLab/source/isaaclab_assets/data/ur5e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 scale=1. 1. 1.
- link wrist_2_link: mass 1.219 -> 1.3; geometry collision mesh filename=file:///home/till/IsaacLab/source/isaaclab_assets/data/ur5e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 scale=1. 1. 1.; visual mesh filename=file:///home/till/IsaacLab/source/isaaclab_assets/data/ur5e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 scale=1. 1. 1.
- link wrist_3_link: mass 0.1879 -> 0.365; geometry collision mesh filename=file:///home/till/IsaacLab/source/isaaclab_assets/data/ur5e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 scale=1. 1. 1.; visual mesh filename=file:///home/till/IsaacLab/source/isaaclab_assets/data/ur5e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 scale=1. 1. 1.
Joints:
- removed joint base_link-base_fixed_joint
- removed joint base_link-base_link_inertia
- removed joint flange-tool0
- removed joint robotiq_base-tcp
- removed joint wrist_3-flange
- removed joint wrist_3-robotiq_base
- added joint base_link_base_link_inertia: type fixed, parent world, child base_link_inertia, origin xyz=0. 0. 0. rpy=0. 0. -3.1415925
- added joint ee_link_root_joint: type fixed, parent wrist_3_link, child ee_link_robotiq_arg2f_base_link, origin xyz=0.0003378 -0.0001611 -0.0070395 rpy=0. 0. 1.5707964
- added joint finger_joint: type revolute, parent ee_link_robotiq_arg2f_base_link, child left_outer_knuckle, origin xyz=0.0001611 -0.0302632 0.0619445 rpy=-2.2957964 0. 3.1415927, axis 1. 0. 0., limit lower=0. upper=0.7 effort=1000. velocity=1.9999999
- added joint gripper_tcp_joint: type fixed, parent ee_link_robotiq_arg2f_base_link, child tcp_link, origin xyz=0.0001611 0.0003378 0.2070395 rpy=0. 0. -1.5707964
- added joint left_inner_finger_joint: type revolute, parent left_outer_finger, child left_inner_finger, origin xyz=-0. 0.0817554 -0.0282203 rpy=-0.725 -0. -0. , axis 1. 0. 0., limit lower=-0.14 upper=0.84 effort=0. velocity=17453.2925199
- added joint left_inner_knuckle_joint: type revolute, parent ee_link_robotiq_arg2f_base_link, child left_inner_knuckle, origin xyz=0.0001611 -0.0123622 0.0684595 rpy=2.2957964 -0. 0.0000001, axis 1. 0. 0., limit lower=-0.84 upper=0.14 effort=0. velocity=17453.2925199
- added joint left_outer_finger_joint: type fixed, parent left_outer_knuckle, child left_outer_finger, origin xyz=-0. -0.0182199 0.0260018 rpy=-0. 0. 3.1415925
- added joint right_inner_finger_joint: type revolute, parent right_outer_finger, child right_inner_finger, origin xyz=0. 0.0817554 -0.0282203 rpy=-0.725 0. -0.0000001, axis 1. 0. 0., limit lower=-0.14 upper=0.84 effort=0. velocity=17453.2925199
- added joint right_inner_knuckle_joint: type revolute, parent ee_link_robotiq_arg2f_base_link, child right_inner_knuckle, origin xyz=0.0001611 0.0130379 0.0684595 rpy=2.2957964 0. 3.1415925, axis 1. 0. 0., limit lower=-0.84 upper=0.14 effort=0. velocity=17453.2925199
- added joint right_outer_finger_joint: type fixed, parent right_outer_knuckle, child right_outer_finger, origin xyz=-0. 0.0182199 0.0260018 rpy=0. 0. 0.
- added joint right_outer_knuckle_joint: type revolute, parent ee_link_robotiq_arg2f_base_link, child right_outer_knuckle, origin xyz=0.0001611 0.0309389 0.0619445 rpy=2.2957964 -0. -3.1415925, axis 1. 0. 0., limit lower=-0.84 upper=0.14 effort=0. velocity=17453.2925199
- added joint ur_root_joint: type fixed, parent ur, child world, origin xyz=0. 0. 0. rpy=0. 0. 0.
- joint elbow_joint: axis 0 0 1 -> 0. 0. 1.; limit lower=-3.141592653589793 upper=3.141592653589793 effort=150.0 velocity=3.141592653589793 -> lower=-3.1415927 upper=3.1415927 effort=150. velocity=3.1415927; origin xyz=-0.425 0 0 rpy=0 0 0 -> xyz=-0.425 0. 0.  rpy=0. 0. 0.
- joint shoulder_lift_joint: axis 0 0 1 -> 0. 0. 1.; limit lower=-6.283185307179586 upper=6.283185307179586 effort=150.0 velocity=3.141592653589793 -> lower=-6.2831853 upper=6.2831853 effort=150. velocity=3.1415927; origin xyz=0 0 0 rpy=1.570796327 0 0 -> xyz=0. 0. 0. rpy=1.5707964 0. 0. 
- joint shoulder_pan_joint: axis 0 0 1 -> 0. 0. 1.; limit lower=-6.283185307179586 upper=6.283185307179586 effort=150.0 velocity=3.141592653589793 -> lower=-6.2831853 upper=6.2831853 effort=150. velocity=3.1415927; origin xyz=0 0 0.1625 rpy=0 0 0 -> xyz=0. 0. 0.1625 rpy=0. 0. 0.
- joint wrist_1_joint: axis 0 0 1 -> 0. 0. 1.; limit lower=-6.283185307179586 upper=6.283185307179586 effort=28.0 velocity=3.141592653589793 -> lower=-6.2831853 upper=6.2831853 effort=28. velocity=3.1415927; origin xyz=-0.3922 0 0.1333 rpy=0 0 0 -> xyz=-0.3922 0. 0.1333 rpy=0. 0. 0.
- joint wrist_2_joint: axis 0 0 1 -> 0. 0. 1.; limit lower=-6.283185307179586 upper=6.283185307179586 effort=28.0 velocity=3.141592653589793 -> lower=-6.2831853 upper=6.2831853 effort=28. velocity=3.1415927; origin xyz=0 -0.0997 -2.044881182297852e-11 rpy=1.570796327 0 0 -> xyz=-0. -0.0997 -0.  rpy=1.5707964 0. 0. 
- joint wrist_3_joint: axis 0 0 1 -> 0. 0. 1.; limit lower=-6.283185307179586 upper=6.283185307179586 effort=28.0 velocity=3.141592653589793 -> lower=-6.2831853 upper=6.2831853 effort=28. velocity=3.1415927; origin xyz=0 0.0996 -2.042830148012698e-11 rpy=1.570796326589793 3.141592653589793 3.141592653589793 -> xyz=0. 0.0996 -0.  rpy=-1.5707964 -0.0000001 0.0000001

Commit message: exchanged Robotiq 2F 140 gripper for newest version, still some kinematics issues that have to be solved

File: source/isaaclab_assets/data/ur5e_dual_setup/ur5e_robotiq_2f_140.urdf (robot description, URDF)
Before this commit: robot ur5e_robotiq_2f_140, 19 links, 18 joints
Links:
- removed link base_link_inertia
- removed link ee_link_robotiq_arg2f_base_link
- removed link ur
- removed link world
- added link World
- added link robotiq_base_link; collision mesh filename=file:///home/till/IsaacLab/source/isaaclab_assets/data/ur5e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 scale=1. 1. 1.; visual mesh filename=file:///home/till/IsaacLab/source/isaaclab_assets/data/ur5e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 scale=1. 1. 1.
- added link ur5e_base_link, mass 4.; collision mesh filename=file:///home/till/IsaacLab/source/isaaclab_assets/data/ur5e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 scale=1. 1. 1.; visual mesh filename=file:///home/till/IsaacLab/source/isaaclab_assets/data/ur5e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 scale=1. 1. 1.
- link forearm_link: mass 2.846 -> 2.2750001
- link left_inner_finger: mass 0.0104003 -> 0.0498344; geometry collision mesh filename=file:///home/till/IsaacLab/source/isaaclab_assets/data/ur5e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 scale=1. 1. 1.; collision mesh filename=file:///home/till/IsaacLab/source/isaaclab_assets/data/ur5e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 scale=1. 1. 1.
- link left_inner_knuckle: mass 0.0271177 -> 0.0681122; geometry collision mesh filename=file:///home/till/IsaacLab/source/isaaclab_assets/data/ur5e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 scale=1. 1. 1.; visual mesh filename=file:///home/till/IsaacLab/source/isaaclab_assets/data/ur5e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 scale=1. 1. 1.
- link left_outer_finger: mass 0.0226142 -> 0.0770643; geometry collision mesh filename=file:///home/till/IsaacLab/source/isaaclab_assets/data/ur5e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 scale=1. 1. 1.; visual mesh filename=file:///home/till/IsaacLab/source/isaaclab_assets/data/ur5e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 scale=1. 1. 1.
- link left_outer_knuckle: mass 0.008532 -> 0.0091633; geometry collision mesh filename=file:///home/till/IsaacLab/source/isaaclab_assets/data/ur5e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 scale=1. 1. 1.; visual mesh filename=file:///home/till/IsaacLab/source/isaaclab_assets/data/ur5e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 scale=1. 1. 1.
- link right_inner_finger: mass 0.0104003 -> 0.0498344; geometry collision mesh filename=file:///home/till/IsaacLab/source/isaaclab_assets/data/ur5e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 scale=1. 1. 1.; collision mesh filename=file:///home/till/IsaacLab/source/isaaclab_assets/data/ur5e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 scale=1. 1. 1.
- link right_inner_knuckle: mass 0.0271177 -> 0.0681122; geometry collision mesh filename=file:///home/till/IsaacLab/source/isaaclab_assets/data/ur5e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 scale=1. 1. 1.; visual mesh filename=file:///home/till/IsaacLab/source/isaaclab_assets/data/ur5e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 scale=1. 1. 1.
- link right_outer_finger: mass 0.0226142 -> 0.0770643; geometry collision mesh filename=file:///home/till/IsaacLab/source/isaaclab_assets/data/ur5e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 scale=1. 1. 1.; visual mesh filename=file:///home/till/IsaacLab/source/isaaclab_assets/data/ur5e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 scale=1. 1. 1.
- link right_outer_knuckle: mass 0.008532 -> 0.0091633; geometry collision mesh filename=file:///home/till/IsaacLab/source/isaaclab_assets/data/ur5e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 scale=1. 1. 1.; visual mesh filename=file:///home/till/IsaacLab/source/isaaclab_assets/data/ur5e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 scale=1. 1. 1.
- link shoulder_link: mass 3.7609999 -> 3.7
- link upper_arm_link: mass 8.0579996 -> 8.3929996
- link wrist_1_link: mass 1.37 -> 1.219
- link wrist_2_link: mass 1.3 -> 1.219
- link wrist_3_link: mass 0.365 -> 0.1879
Joints:
- removed joint base_link_base_link_inertia
- removed joint ee_link_root_joint
- removed joint left_inner_finger_joint
- removed joint right_inner_finger_joint
- removed joint ur_root_joint
- added joint AssemblerFixedJoint: type fixed, parent wrist_3_link, child robotiq_base_link, origin xyz=-0. -0. -0. rpy=0. 0. 0.
- added joint left_inner_finger_pad_joint: type revolute, parent left_outer_finger, child left_inner_finger, origin xyz=0 0.0454 0.0125 rpy=0 0 0, axis 0 0 1, limit lower=-3.1415 upper=3.1415 effort=100 velocity=2.0, mimic joint=finger_joint multiplier=-1.0 offset=0.0
- added joint right_inner_finger_pad_joint: type revolute, parent right_outer_finger, child right_inner_finger, origin xyz=0.045 -0.012 0 rpy=0 0 0, axis 0 0 1, limit lower=-3.1415 upper=3.1415 effort=100 velocity=2.0, mimic joint=finger_joint multiplier=-1.0 offset=0.0
- added joint root_joint: type fixed, parent World, child ur5e_base_link, origin xyz=0. 0. 0. rpy=0. 0. 0.
- joint finger_joint: axis 1. 0. 0. -> 0 0 1; limit lower=0. upper=0.7 effort=1000. velocity=1.9999999 -> lower=0 upper=1.308996 effort=1000 velocity=2.0; origin xyz=0.0001611 -0.0302632 0.0619445 rpy=-2.2957964 0. 3.1415927 -> xyz=0 -0.0306 0.0546 rpy=1.5707 0 -1.5707; parent ee_link_robotiq_arg2f_base_link -> robotiq_base_link
- joint gripper_tcp_joint: origin xyz=0.0001611 0.0003378 0.2070395 rpy=0. 0. -1.5707964 -> xyz=0. 0. 0.2 rpy=-3.1415927 -1.5707964 0. ; parent ee_link_robotiq_arg2f_base_link -> robotiq_base_link
- joint left_inner_knuckle_joint: axis 1. 0. 0. -> 0 0 1; limit lower=-0.84 upper=0.14 effort=0. velocity=17453.2925199 -> lower=0 upper=1.308996 effort=100 velocity=2.0; mimic (none) -> joint=finger_joint multiplier=1.0 offset=0.0; origin xyz=0.0001611 -0.0123622 0.0684595 rpy=2.2957964 -0. 0.0000001 -> xyz=0 -0.0127 0.0614 rpy=1.5707 0 -1.5707; parent ee_link_robotiq_arg2f_base_link -> robotiq_base_link
- joint left_outer_finger_joint: origin xyz=-0. -0.0182199 0.0260018 rpy=-0. 0. 3.1415925 -> xyz=0 0.0315 -0.0041 rpy=0 0 0
- joint right_inner_knuckle_joint: axis 1. 0. 0. -> 0. 0. 1.; limit lower=-0.84 upper=0.14 effort=0. velocity=17453.2925199 -> lower=0.0 upper=1.308996 effort=10. velocity=2.268928; mimic (none) -> joint=finger_joint multiplier=-1.0 offset=0.0; origin xyz=0.0001611 0.0130379 0.0684595 rpy=2.2957964 0. 3.1415925 -> xyz=0. 0.0127 0.061178 rpy=-1.5707964 0. 1.5707964; parent ee_link_robotiq_arg2f_base_link -> robotiq_base_link
- joint right_outer_finger_joint: axis (none) -> 0. 0. 1.; origin xyz=-0. 0.0182199 0.0260018 rpy=0. 0. 0. -> xyz=0.0314249 -0.0045322 0.  rpy=-3.1415927 0. -3.1415927
- joint right_outer_knuckle_joint: axis 1. 0. 0. -> 0. 0. 1.; limit lower=-0.84 upper=0.14 effort=0. velocity=17453.2925199 -> lower=0. upper=1.308996 effort=10. velocity=2.268928; mimic (none) -> joint=finger_joint multiplier=1.0 offset=0.0; origin xyz=0.0001611 0.0309389 0.0619445 rpy=2.2957964 -0. -3.1415925 -> xyz=0. 0.0306011 0.0546625 rpy=1.5707964 0. 1.5707964; parent ee_link_robotiq_arg2f_base_link -> robotiq_base_link
- joint shoulder_pan_joint: origin xyz=0. 0. 0.1625 rpy=0. 0. 0. -> xyz=0. 0. 0.1625 rpy=0. 0. -3.1415925; parent base_link_inertia -> ur5e_base_link

Commit message: setup update - toolchanger included, back to old gripper
current bug: arm drifts if gripper is opened using controller

File: source/isaaclab_assets/data/ur5e_dual_setup/ur5e_robotiq_2f_140.urdf (robot description, URDF)
Before this commit: robot ur5e_robotiq_2f_140, 18 links, 17 joints
Links:
- removed link robotiq_base_link
- added link pdc_connector_link; collision mesh filename=file:///home/till/IsaacLab/source/isaaclab_assets/data/ur5e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 scale=1. 1. 1.; visual mesh filename=file:///home/till/IsaacLab/source/isaaclab_assets/data/ur5e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 scale=1. 1. 1.
- added link robotiq_2f_140_robotiq_arg2f_base_link, mass 0.22652; collision mesh filename=file:///home/till/IsaacLab/source/isaaclab_assets/data/ur5e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 scale=1. 1. 1.; visual mesh filename=file:///home/till/IsaacLab/source/isaaclab_assets/data/ur5e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 scale=1. 1. 1.
- added link tool_changer_robot_side_link; collision mesh filename=file:///home/till/IsaacLab/source/isaaclab_assets/data/ur5e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 scale=1. 1. 1.; visual mesh filename=file:///home/till/IsaacLab/source/isaaclab_assets/data/ur5e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 scale=1. 1. 1.
- added link tool_changer_tool_side_link; collision mesh filename=file:///home/till/IsaacLab/source/isaaclab_assets/data/ur5e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 scale=1. 1. 1.; visual mesh filename=file:///home/till/IsaacLab/source/isaaclab_assets/data/ur5e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 scale=1. 1. 1.
- link left_inner_finger: mass 0.0498344 -> 0.0104003; geometry collision box size=0.03 0.07 0.0075; collision mesh filename=file:///home/till/IsaacLab/source/isaaclab_assets/data/ur5e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 scale=1. 1. 1.
- link left_inner_knuckle: mass 0.0681122 -> 0.0271177; geometry collision mesh filename=file:///home/till/IsaacLab/source/isaaclab_assets/data/ur5e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 scale=1. 1. 1.; visual mesh filename=file:///home/till/IsaacLab/source/isaaclab_assets/data/ur5e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 scale=1. 1. 1.
- link left_outer_finger: mass 0.0770643 -> 0.0226142; geometry collision mesh filename=file:///home/till/IsaacLab/source/isaaclab_assets/data/ur5e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 scale=1. 1. 1.; visual mesh filename=file:///home/till/IsaacLab/source/isaaclab_assets/data/ur5e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 scale=1. 1. 1.
- link left_outer_knuckle: mass 0.0091633 -> 0.008532; geometry collision mesh filename=file:///home/till/IsaacLab/source/isaaclab_assets/data/ur5e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 scale=1. 1. 1.; visual mesh filename=file:///home/till/IsaacLab/source/isaaclab_assets/data/ur5e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 scale=1. 1. 1.
- link right_inner_finger: mass 0.0498344 -> 0.0104003; geometry collision box size=0.03 0.07 0.0075; collision mesh filename=file:///home/till/IsaacLab/source/isaaclab_assets/data/ur5e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 scale=1. 1. 1.
- link right_inner_knuckle: mass 0.0681122 -> 0.0271177; geometry collision mesh filename=file:///home/till/IsaacLab/source/isaaclab_assets/data/ur5e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 scale=1. 1. 1.; visual mesh filename=file:///home/till/IsaacLab/source/isaaclab_assets/data/ur5e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 scale=1. 1. 1.
- link right_outer_finger: mass 0.0770643 -> 0.0226142; geometry collision mesh filename=file:///home/till/IsaacLab/source/isaaclab_assets/data/ur5e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 scale=1. 1. 1.; visual mesh filename=file:///home/till/IsaacLab/source/isaaclab_assets/data/ur5e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 scale=1. 1. 1.
- link right_outer_knuckle: mass 0.0091633 -> 0.008532; geometry collision mesh filename=file:///home/till/IsaacLab/source/isaaclab_assets/data/ur5e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 scale=1. 1. 1.; visual mesh filename=file:///home/till/IsaacLab/source/isaaclab_assets/data/ur5e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 scale=1. 1. 1.
Joints:
- removed joint AssemblerFixedJoint
- removed joint gripper_tcp_joint
- removed joint left_inner_finger_pad_joint
- removed joint right_inner_finger_pad_joint
- added joint gripper_base_tcp_joint: type fixed, parent robotiq_2f_140_robotiq_arg2f_base_link, child tcp_link, origin xyz=0. -0. 0.2 rpy=1.5707964 -0. 1.5707964
- added joint left_inner_finger_joint: type revolute, parent left_outer_finger, child left_inner_finger, origin xyz=0. 0.0817554 -0.0282203 rpy=-0.725 0. 0. , axis 1. 0. 0., limit lower=-0.14 upper=0.84 effort=0. velocity=17453.2925199
- added joint pdc_gripper_joint: type fixed, parent pdc_connector_link, child robotiq_2f_140_robotiq_arg2f_base_link, origin xyz=-0. 0.0139 0.  rpy=-1.5519305 -1.5707947 -0.0188656
- added joint right_inner_finger_joint: type revolute, parent right_outer_finger, child right_inner_finger, origin xyz=0. 0.0817554 -0.0282203 rpy=-0.725 0. 0. , axis 1. 0. 0., limit lower=-0.14 upper=0.84 effort=0. velocity=17453.2925199
- added joint robot_gripper_joint: type fixed, parent wrist_3_link, child tool_changer_robot_side_link, origin xyz=-0. -0. -0.0000001 rpy=-1.5707963 -1.5707964 0. 
- added joint tool_changer_joint: type fixed, parent tool_changer_robot_side_link, child tool_changer_tool_side_link, origin xyz=0.0243747 -0.0000721 0.0004423 rpy=-3.1415925 -0.0006422 -1.570829 
- added joint tool_changer_tool_pdc_joint: type fixed, parent tool_changer_tool_side_link, child pdc_connector_link, origin xyz=-0.0000724 -0.0001253 0.0004423 rpy=3.1415925 -0.0006406 -0.0000326
- joint finger_joint: axis 0 0 1 -> 1. 0. 0.; limit lower=0 upper=1.308996 effort=1000 velocity=2.0 -> lower=0. upper=0.7 effort=1000. velocity=1.9999999; origin xyz=0 -0.0306 0.0546 rpy=1.5707 0 -1.5707 -> xyz=0. -0.030601 0.054905 rpy=-2.2957964 -0. -3.1415925; parent robotiq_base_link -> robotiq_2f_140_robotiq_arg2f_base_link
- joint left_inner_knuckle_joint: axis 0 0 1 -> 1. 0. 0.; limit lower=0 upper=1.308996 effort=100 velocity=2.0 -> lower=-0.84 upper=0.14 effort=0. velocity=17453.2925199; mimic joint=finger_joint multiplier=1.0 offset=0.0 -> (none); origin xyz=0 -0.0127 0.0614 rpy=1.5707 0 -1.5707 -> xyz=0. -0.0127 0.06142 rpy=2.2957964 0. 0.0000001; parent robotiq_base_link -> robotiq_2f_140_robotiq_arg2f_base_link
- joint left_outer_finger_joint: origin xyz=0 0.0315 -0.0041 rpy=0 0 0 -> xyz=0. -0.01822 0.0260018 rpy=-0. 0. 3.1415927
- joint right_inner_knuckle_joint: axis 0. 0. 1. -> 1. 0. 0.; limit lower=0.0 upper=1.308996 effort=10. velocity=2.268928 -> lower=-0.84 upper=0.14 effort=0. velocity=17453.2925199; mimic joint=finger_joint multiplier=-1.0 offset=0.0 -> (none); origin xyz=0. 0.0127 0.061178 rpy=-1.5707964 0. 1.5707964 -> xyz=-0. 0.0127 0.06142 rpy=2.2957964 -0. 3.1415927; parent robotiq_base_link -> robotiq_2f_140_robotiq_arg2f_base_link
- joint right_outer_finger_joint: axis 0. 0. 1. -> (none); origin xyz=0.0314249 -0.0045322 0.  rpy=-3.1415927 0. -3.1415927 -> xyz=0. 0.01822 0.0260018 rpy=0. 0. 0.
- joint right_outer_knuckle_joint: axis 0. 0. 1. -> 1. 0. 0.; limit lower=0. upper=1.308996 effort=10. velocity=2.268928 -> lower=-0.84 upper=0.14 effort=0. velocity=17453.2925199; mimic joint=finger_joint multiplier=1.0 offset=0.0 -> (none); origin xyz=0. 0.0306011 0.0546625 rpy=1.5707964 0. 1.5707964 -> xyz=-0. 0.030601 0.054905 rpy=2.2957964 -0. -3.1415925; parent robotiq_base_link -> robotiq_2f_140_robotiq_arg2f_base_link
