Commit message: fixed drifting gripper

File: source/isaaclab_assets/data/ur5e_dual_setup/ur5e_robotiq_2f_140.urdf (robot description, URDF)
Before this commit: robot ur5e_robotiq_2f_140_toolchanger_c, 21 links, 20 joints
Links:
- added link left_inner_finger_pad; collision box size=0.03 0.07 0.0075; visual box size=0.027 0.065 0.0075
- added link right_inner_finger_pad; collision box size=0.03 0.07 0.0075; visual box size=0.027 0.065 0.0075
- link left_inner_finger: mass 0.0104003 -> 0.0104003125914103; geometry visual mesh filename=file:///home/till/IsaacLab/source/isaaclab_assets/data/ur5e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 scale=1. 1. 1.
- link left_inner_knuckle: mass 0.0271177 -> 0.0271177346495152; geometry visual mesh filename=file:///home/till/IsaacLab/source/isaaclab_assets/data/ur5e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 scale=1. 1. 1.
- link left_outer_finger: mass 0.0226142 -> 0.022614240507152; geometry visual mesh filename=file:///home/till/IsaacLab/source/isaaclab_assets/data/ur5e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 scale=1. 1. 1.
- link left_outer_knuckle: mass 0.008532 -> 0.00853198276973456; geometry visual mesh filename=file:///home/till/IsaacLab/source/isaaclab_assets/data/ur5e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 scale=1. 1. 1.
- link right_inner_finger: mass 0.0104003 -> 0.0104003125914103; geometry visual mesh filename=file:///home/till/IsaacLab/source/isaaclab_assets/data/ur5e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 scale=1. 1. 1.
- link right_inner_knuckle: mass 0.0271177 -> 0.0271177346495152; geometry visual mesh filename=file:///home/till/IsaacLab/source/isaaclab_assets/data/ur5e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 scale=1. 1. 1.
- link right_outer_finger: mass 0.0226142 -> 0.022614240507152; geometry visual mesh filename=file:///home/till/IsaacLab/source/isaaclab_assets/data/ur5e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 scale=1. 1. 1.
- link right_outer_knuckle: mass 0.008532 -> 0.00853198276973456; geometry visual mesh filename=file:///home/till/IsaacLab/source/isaaclab_assets/data/ur5e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 scale=1. 1. 1.
- link robotiq_2f_140_robotiq_arg2f_base_link: geometry collision mesh filename=file:///home/till/IsaacLab/source/isaaclab_assets/data/ur5e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 scale=1. 1. 1.; visual mesh filename=file:///home/till/IsaacLab/source/isaaclab_assets/data/ur5e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 scale=1. 1. 1.
Joints:
- added joint left_inner_finger_pad_joint: type fixed, parent left_inner_finger, child left_inner_finger_pad, origin xyz=0. 0.0457554015893473 -0.0272203446692936 rpy=0 0 0, axis 0 0 1
- added joint right_inner_finger_pad_joint: type fixed, parent right_inner_finger, child right_inner_finger_pad, origin xyz=0. 0.0457554015893473 -0.0272203446692936 rpy=0 0 0, axis 0 0 1
- joint elbow_joint: origin xyz=-0.425 0. 0.  rpy=0. 0. 0. -> xyz=-0.425 0. 0. rpy=0. 0. 0.
- joint finger_joint: axis 1. 0. 0. -> -1 0 0; limit lower=0. upper=0.7 effort=1000. velocity=1.9999999 -> lower=0 upper=0.7 effort=1000 velocity=2.0; origin xyz=0. -0.030601 0.054905 rpy=-2.2957964 -0. -3.1415925 -> xyz=0. -0.030601 0.054905 rpy=2.2957963267948966 0 0
- joint gripper_base_tcp_joint: origin xyz=0. -0. 0.2 rpy=1.5707964 -0. 1.5707964 -> xyz=0. 0. 0.2 rpy=1.5707964 0. 1.5707964
- joint left_inner_finger_joint: axis 1. 0. 0. -> 1 0 0; limit lower=-0.14 upper=0.84 effort=0. velocity=17453.2925199 -> lower=-0.8757 upper=0.8757 effort=1000 velocity=2.0; mimic (none) -> joint=finger_joint multiplier=1 offset=0; origin xyz=0. 0.0817554 -0.0282203 rpy=-0.725 0. 0.  -> xyz=0. 0.0817554015893473 -0.0282203446692936 rpy=-0.725 0 0
- joint left_inner_knuckle_joint: axis 1. 0. 0. -> 1 0 0; limit lower=-0.84 upper=0.14 effort=0. velocity=17453.2925199 -> lower=-0.8757 upper=0.8757 effort=1000 velocity=2.0; mimic (none) -> joint=finger_joint multiplier=-1 offset=0; origin xyz=0. -0.0127 0.06142 rpy=2.2957964 0. 0.0000001 -> xyz=0. -0.0127 0.06142 rpy=2.2957963267948966 0 0.0
- joint left_outer_finger_joint: axis (none) -> 1 0 0; origin xyz=0. -0.01822 0.0260018 rpy=-0. 0. 3.1415927 -> xyz=0. 0.01821998610742 0.0260018192872234 rpy=0 0 0
- joint pdc_gripper_joint: origin xyz=-0. 0.0139 0.  rpy=-1.5519305 -1.5707947 -0.0188656 -> xyz=0. 0.0139 0. rpy=-1.5519305 -1.5707947 -0.0188656
- joint right_inner_finger_joint: axis 1. 0. 0. -> 1 0 0; limit lower=-0.14 upper=0.84 effort=0. velocity=17453.2925199 -> lower=-0.8757 upper=0.8757 effort=1000 velocity=2.0; mimic (none) -> joint=finger_joint multiplier=1 offset=0; origin xyz=0. 0.0817554 -0.0282203 rpy=-0.725 0. 0.  -> xyz=0. 0.0817554015893473 -0.0282203446692936 rpy=-0.725 0 0
- joint right_inner_knuckle_joint: axis 1. 0. 0. -> 1 0 0; limit lower=-0.84 upper=0.14 effort=0. velocity=17453.2925199 -> lower=-0.8757 upper=0.8757 effort=1000 velocity=2.0; mimic (none) -> joint=finger_joint multiplier=-1 offset=0; origin xyz=-0. 0.0127 0.06142 rpy=2.2957964 -0. 3.1415927 -> xyz=0. 0.0127 0.06142 rpy=2.2957963267948966 0 -3.141592653589793
- joint right_outer_finger_joint: axis (none) -> 1 0 0; origin xyz=0. 0.01822 0.0260018 rpy=0. 0. 0. -> xyz=0. 0.01821998610742 0.0260018192872234 rpy=0 0 0
- joint right_outer_knuckle_joint: axis 1. 0. 0. -> 1 0 0; limit lower=-0.84 upper=0.14 effort=0. velocity=17453.2925199 -> lower=-0.725 upper=0.725 effort=1000 velocity=2.0; mimic (none) -> joint=finger_joint multiplier=-1 offset=0; origin xyz=-0. 0.030601 0.054905 rpy=2.2957964 -0. -3.1415925 -> xyz=0. 0.030601 0.054905 rpy=2.2957963267948966 0 3.141592653589793
- joint robot_gripper_joint: origin xyz=-0. -0. -0.0000001 rpy=-1.5707963 -1.5707964 0.  -> xyz=0. 0. -0.0000001 rpy=-1.5707963 -1.5707964 0.
- joint shoulder_lift_joint: origin xyz=0. 0. 0. rpy=1.5707964 0. 0.  -> xyz=0. 0. 0. rpy=1.5707964 0. 0.
- joint tool_changer_joint: origin xyz=0.0243747 -0.0000721 0.0004423 rpy=-3.1415925 -0.0006422 -1.570829  -> xyz=0.0243747 -0.0000721 0.0004423 rpy=-3.1415925 -0.0006422 -1.570829
- joint wrist_2_joint: origin xyz=-0. -0.0997 -0.  rpy=1.5707964 0. 0.  -> xyz=0. -0.0997 0. rpy=1.5707964 0. 0.
- joint wrist_3_joint: origin xyz=0. 0.0996 -0.  rpy=-1.5707964 -0.0000001 0.0000001 -> xyz=0. 0.0996 0. rpy=-1.5707964 -0.0000001 0.0000001

Commit message: teleoperation first working prototype

File: source/isaaclab_assets/data/ur5e_dual_setup/ur5e_robotiq_2f_140.urdf (robot description, URDF)
Before this commit: robot ur5e_robotiq_2f_140_toolchanger_c, 23 links, 22 joints
Links:
- link left_inner_finger: geometry collision mesh filename=file:///home/till/IsaacLab/source/isaaclab_assets/data/ur5e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 scale=1. 1. 1.; visual mesh filename=file:///home/till/IsaacLab/source/isaaclab_assets/data/ur5e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 scale=1. 1. 1.
- link left_inner_knuckle: geometry collision mesh filename=file:///home/till/IsaacLab/source/isaaclab_assets/data/ur5e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 scale=1. 1. 1.; visual mesh filename=file:///home/till/IsaacLab/source/isaaclab_assets/data/ur5e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 scale=1. 1. 1.
- link left_outer_finger: geometry collision mesh filename=file:///home/till/IsaacLab/source/isaaclab_assets/data/ur5e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 scale=1. 1. 1.; visual mesh filename=file:///home/till/IsaacLab/source/isaaclab_assets/data/ur5e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 scale=1. 1. 1.
- link left_outer_knuckle: geometry collision mesh filename=file:///home/till/IsaacLab/source/isaaclab_assets/data/ur5e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 scale=1. 1. 1.; visual mesh filename=file:///home/till/IsaacLab/source/isaaclab_assets/data/ur5e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 scale=1. 1. 1.
- link right_inner_finger: geometry collision mesh filename=file:///home/till/IsaacLab/source/isaaclab_assets/data/ur5e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 scale=1. 1. 1.; visual mesh filename=file:///home/till/IsaacLab/source/isaaclab_assets/data/ur5e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 scale=1. 1. 1.
- link right_inner_knuckle: geometry collision mesh filename=file:///home/till/IsaacLab/source/isaaclab_assets/data/ur5e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 scale=1. 1. 1.; visual mesh filename=file:///home/till/IsaacLab/source/isaaclab_assets/data/ur5e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 scale=1. 1. 1.
- link right_outer_finger: geometry collision mesh filename=file:///home/till/IsaacLab/source/isaaclab_assets/data/ur5e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 scale=1. 1. 1.; visual mesh filename=file:///home/till/IsaacLab/source/isaaclab_assets/data/ur5e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 scale=1. 1. 1.
- link right_outer_knuckle: geometry collision mesh filename=file:///home/till/IsaacLab/source/isaaclab_assets/data/ur5e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 scale=1. 1. 1.; visual mesh filename=file:///home/till/IsaacLab/source/isaaclab_assets/data/ur5e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 scale=1. 1. 1.

Commit message: updated control frequency and tuned simulation to match real robot

File: source/isaaclab_assets/data/ur5e_dual_setup/ur5e_robotiq_2f_140.urdf (robot description, URDF)
Before this commit: robot ur5e_robotiq_2f_140_toolchanger_c, 23 links, 22 joints
Joints:
- joint elbow_joint: limit lower=-3.1415927 upper=3.1415927 effort=150. velocity=3.1415927 -> lower=-6.2831853 upper=6.2831853 effort=150. velocity=3.1415927
